Commit message: launch gazebo moveit seperately, use velocity_controller and diff_dri…  …

File: urdf/simple_robot.urdf (robot description, URDF)
Before this commit: robot simple_robot, 13 links, 12 joints
Links:
- link mobile_base_link: mass 50 -> None
- link wheel_left_link: mass 5 -> 0.5
- link wheel_right_link: mass 5 -> 0.5

File: urdf/simple_robot.urdf.xacro (robot description, xacro)
@@ -29,5 +29,5 @@
   </xacro:macro>
   <xacro:include filename="$(find simple_robot_description)/urdf/materials.urdf.xacro"/>
-  <xacro:include filename="$(find simple_robot_description)/urdf/sr.gazebo"/>
+  <xacro:include filename="$(find simple_robot_description)/urdf/simple_robot.gazebo"/>
   <xacro:include filename="$(find simple_robot_description)/urdf/common.xacro"/>
   <robotBaseFrame>mobile_base_link</robotBaseFrame>
